File: hardware/adapters/core2021-hf-m-rev-a/core2021-hf-m-rev-a.kicad_sch (KiCad schematic)
At the start: 13 parts, among them J1 TSW-110-07-G-S, J2 TSW-108-07-G-S, J3 SSQ-108-01-G-S, J4 SSQ-108-01-G-S, U1 Core2021-HF-M plug-in, U2 AP2112K-3.3TRG1

Commit message: Add configurable SPI source termination
Parts:
- added R3: 22, Resistor_SMD:R_0603_1608Metric, symbol RadioLab:Resistor_value_only
Connections:
- net SPI_MISO: now also R3.2; no longer J4.3, U1.11 (MISO)
- new net SPI_MISO_SRC: J4.3, R3.1, U1.11 (MISO)
Other:
- note added: "MISO: source -> 22R -> slot A7. Fit 0R option; scope/IBIS verify. Place at module output/socket, before shared bus. No long stubs."

Commit message: Add routed Rev-A PCB layouts and board review
Parts:
- added TP1: SPI_SCK, RadioLab:Probe_Pad_D1.0mm, symbol RadioLab:Probe_point
- added TP10: AUX0, RadioLab:Probe_Pad_D1.0mm, symbol RadioLab:Probe_point
- added TP11: OUT_3V3, RadioLab:Probe_Pad_D1.0mm, symbol RadioLab:Probe_point
- added TP12: REG_GND, RadioLab:Probe_Pad_D1.0mm, symbol RadioLab:Probe_point
- added TP13: EN_5V, RadioLab:Probe_Pad_D1.0mm, symbol RadioLab:Probe_point
- added TP14: MOD_3V3, RadioLab:Probe_Pad_D1.0mm, symbol RadioLab:Probe_point
- added TP15: MOD_GND, RadioLab:Probe_Pad_D1.0mm, symbol RadioLab:Probe_point
- added TP2: SPI_MOSI, RadioLab:Probe_Pad_D1.0mm, symbol RadioLab:Probe_point
- added TP3: SPI_MISO, RadioLab:Probe_Pad_D1.0mm, symbol RadioLab:Probe_point
- added TP4: CS_N, RadioLab:Probe_Pad_D1.0mm, symbol RadioLab:Probe_point
- added TP5: RESET_N, RadioLab:Probe_Pad_D1.0mm, symbol RadioLab:Probe_point
- added TP6: BUSY, RadioLab:Probe_Pad_D1.0mm, symbol RadioLab:Probe_point
- added TP7: IRQ, RadioLab:Probe_Pad_D1.0mm, symbol RadioLab:Probe_point
- added TP8: IN_5V, RadioLab:Probe_Pad_D1.0mm, symbol RadioLab:Probe_point
- added TP9: CLIP_GND, TestPoint:TestPoint_Keystone_5010-5014_Multipurpose, symbol RadioLab:Probe_point
Connections:
- net AUX0: now also TP10.1 (PROBE)
- net BUSY: now also TP6.1 (PROBE)
- net CS_N: now also TP4.1 (PROBE)
- net GND: now also TP12.1 (PROBE), TP15.1 (PROBE), TP9.1 (PROBE)
- net IRQ: now also TP7.1 (PROBE)
- net RADIO_3V3: now also TP11.1 (PROBE), TP14.1 (PROBE)
- net RESET_N: now also TP5.1 (PROBE)
- net SLOT_5V: now also TP13.1 (PROBE), TP8.1 (PROBE)
- net SPI_MISO: now also TP3.1 (PROBE)
- net SPI_MOSI: now also TP2.1 (PROBE)
- net SPI_SCK: now also TP1.1 (PROBE)
Other:
- note added: "KEYED SLOT: H1 engages the carrier M3 x 25 post before electrical contact. All headers and passives factory fitted. No user soldering or antenna-selector rework. Power declarations describe power arriving through the slot and buck output after L1. Layout authorized; no fabrication release. See DESIGN_REVIEW.md."
- note added: "REV A LAYOUT REVIEW. NOT FOR FABRICATION."
- note removed: "KEYED SLOT: H1 engages the carrier M3 x 25 post before electrical contact. All headers and passives factory fitted. No user soldering or antenna-selector rework. Power declarations describe power arriving through the slot and buck output after L1. No PCB layout is authorized. Footprint and assembly evidence: see DESIGN_REVIEW.md."
- note removed: "REV A SCHEMATIC REVIEW. NO PCB LAYOUT OR FABRICATION RELEASE."
