File: hardware/carrier-rev-a/carrier-rev-a.kicad_sch (KiCad schematic)
At the start: 59 parts, among them J1 SSQ-110-01-G-S, J10 SSQ-120-01-G-S, J11 SSQ-120-01-G-S, J2 SSQ-108-01-G-S, J3 SSQ-110-01-G-S, J4 SSQ-108-01-G-S, J5 SSQ-110-01-G-S, J6 SSQ-108-01-G-S, J7 SSQ-110-01-G-S, J8 SSQ-108-01-G-S, J9 5 V / 4 A INPUT, Q1 DMG2305UX-7, U1 Pico 2 with headers, SC1632, U2 TPS259470LRPWR, U3 AP2112K-3.3TRG1, U4 MCP23S17-E/SO, U5 SN74LVC8T245PWR, U6 SN74LVC8T245PWR, U7 SN74LVC1T45DBVR

Commit message: Add configurable SPI source termination
Parts:
- added R20, R21, R22: 22, Resistor_SMD:R_0603_1608Metric, symbol RadioLab:Resistor_value_only
Connections:
- net SPI_MISO: now also R22.2; no longer U4.14 (SO)
- net SPI_MOSI: now also R21.2; no longer U5.20 (B2)
- net SPI_SCK: now also R20.2; no longer U5.21 (B1)
- new net EXP_MISO_SRC: R22.1, U4.14 (SO)
- new net SPI_MOSI_SRC: R21.1, U5.20 (B2)
- new net SPI_SCK_SRC: R20.1, U5.21 (B1)
Other:
- note added: "R20/R21: immediately after U5 SCK/MOSI outputs. R22: at U4 SO before shared MISO. 22R initial; 0R population option. Verify by oscilloscope/IBIS. No long stubs. Each radio card has its own MISO source resistor before slot A7."

Commit message: Add routed Rev-A PCB layouts and board review
Parts:
- added TP1: S1_5V, RadioLab:Probe_Pad_D1.0mm, symbol RadioLab:Probe_point
- added TP10: S2_CS_N, RadioLab:Probe_Pad_D1.0mm, symbol RadioLab:Probe_point
- added TP11: S2_BUSY, RadioLab:Probe_Pad_D1.0mm, symbol RadioLab:Probe_point
- added TP12: S2_IRQ, RadioLab:Probe_Pad_D1.0mm, symbol RadioLab:Probe_point
- added TP13: S2_RESET_N, RadioLab:Probe_Pad_D1.0mm, symbol RadioLab:Probe_point
- added TP14: S2_GND, TestPoint:TestPoint_Keystone_5010-5014_Multipurpose, symbol RadioLab:Probe_point
- added TP15: S3_5V, RadioLab:Probe_Pad_D1.0mm, symbol RadioLab:Probe_point
- added TP16: S3_CS_N, RadioLab:Probe_Pad_D1.0mm, symbol RadioLab:Probe_point
- added TP17: S3_BUSY, RadioLab:Probe_Pad_D1.0mm, symbol RadioLab:Probe_point
- added TP18: S3_IRQ, RadioLab:Probe_Pad_D1.0mm, symbol RadioLab:Probe_point
- added TP19: S3_RESET_N, RadioLab:Probe_Pad_D1.0mm, symbol RadioLab:Probe_point
- added TP2: S1_CS_N, RadioLab:Probe_Pad_D1.0mm, symbol RadioLab:Probe_point
- added TP20: S3_TX_EN, RadioLab:Probe_Pad_D1.0mm, symbol RadioLab:Probe_point
- added TP21: S3_RX_EN, RadioLab:Probe_Pad_D1.0mm, symbol RadioLab:Probe_point
- added TP22: S3_GND, TestPoint:TestPoint_Keystone_5010-5014_Multipurpose, symbol RadioLab:Probe_point
- added TP23: S4_5V, RadioLab:Probe_Pad_D1.0mm, symbol RadioLab:Probe_point
- added TP24: S4_CS_N, RadioLab:Probe_Pad_D1.0mm, symbol RadioLab:Probe_point
- added TP25: S4_BUSY, RadioLab:Probe_Pad_D1.0mm, symbol RadioLab:Probe_point
- added TP26: S4_IRQ, RadioLab:Probe_Pad_D1.0mm, symbol RadioLab:Probe_point
- added TP27: S4_RESET_N, RadioLab:Probe_Pad_D1.0mm, symbol RadioLab:Probe_point
- added TP28: S4_TX_EN, RadioLab:Probe_Pad_D1.0mm, symbol RadioLab:Probe_point
- added TP29: S4_RX_EN, RadioLab:Probe_Pad_D1.0mm, symbol RadioLab:Probe_point
- added TP3: S1_BUSY, RadioLab:Probe_Pad_D1.0mm, symbol RadioLab:Probe_point
- added TP30: S4_GND, TestPoint:TestPoint_Keystone_5010-5014_Multipurpose, symbol RadioLab:Probe_point
- added TP31: IN_5V, RadioLab:Probe_Pad_D1.0mm, symbol RadioLab:Probe_point
- added TP32: BUS_5V, RadioLab:Probe_Pad_D1.0mm, symbol RadioLab:Probe_point
- added TP33: VBUS, RadioLab:Probe_Pad_D1.0mm, symbol RadioLab:Probe_point
- added TP34: VSYS, RadioLab:Probe_Pad_D1.0mm, symbol RadioLab:Probe_point
- added TP35: PICO_3V3, RadioLab:Probe_Pad_D1.0mm, symbol RadioLab:Probe_point
- added TP36: IOREF_3V3, RadioLab:Probe_Pad_D1.0mm, symbol RadioLab:Probe_point
- added TP37: UVLO, RadioLab:Probe_Pad_D1.0mm, symbol RadioLab:Probe_point
- added TP38: OVLO, RadioLab:Probe_Pad_D1.0mm, symbol RadioLab:Probe_point
- added TP39: DVDT, RadioLab:Probe_Pad_D1.0mm, symbol RadioLab:Probe_point
- added TP4: S1_IRQ, RadioLab:Probe_Pad_D1.0mm, symbol RadioLab:Probe_point
- added TP40: ILIM, RadioLab:Probe_Pad_D1.0mm, symbol RadioLab:Probe_point
- added TP41: EXP_CS, RadioLab:Probe_Pad_D1.0mm, symbol RadioLab:Probe_point
- added TP42: EXP_RST, RadioLab:Probe_Pad_D1.0mm, symbol RadioLab:Probe_point
- added TP43: OE_N, RadioLab:Probe_Pad_D1.0mm, symbol RadioLab:Probe_point
- added TP44: P_SCK, RadioLab:Probe_Pad_D1.0mm, symbol RadioLab:Probe_point
- added TP45: P_MOSI, RadioLab:Probe_Pad_D1.0mm, symbol RadioLab:Probe_point
- added TP46: P_MISO, RadioLab:Probe_Pad_D1.0mm, symbol RadioLab:Probe_point
- added TP47: SCK, RadioLab:Probe_Pad_D1.0mm, symbol RadioLab:Probe_point
- added TP48: MOSI, RadioLab:Probe_Pad_D1.0mm, symbol RadioLab:Probe_point
- added TP49: MISO, RadioLab:Probe_Pad_D1.0mm, symbol RadioLab:Probe_point
- added TP5: S1_RESET_N, RadioLab:Probe_Pad_D1.0mm, symbol RadioLab:Probe_point
- added TP50: ENTRY_GND, TestPoint:TestPoint_Keystone_5010-5014_Multipurpose, symbol RadioLab:Probe_point
- added TP51: U3_GND, RadioLab:Probe_Pad_D1.0mm, symbol RadioLab:Probe_point
- added TP6: S1_TX_EN, RadioLab:Probe_Pad_D1.0mm, symbol RadioLab:Probe_point
- added TP7: S1_RX_EN, RadioLab:Probe_Pad_D1.0mm, symbol RadioLab:Probe_point
- added TP8: S1_GND, TestPoint:TestPoint_Keystone_5010-5014_Multipurpose, symbol RadioLab:Probe_point
- added TP9: S2_5V, RadioLab:Probe_Pad_D1.0mm, symbol RadioLab:Probe_point
Connections:
- net DVDT: now also TP39.1 (PROBE)
- net EXP_CS_N: now also TP41.1 (PROBE)
- net EXP_RESET_N: now also TP42.1 (PROBE)
- net EXT_5V: now also TP31.1 (PROBE)
- net GND: now also TP14.1 (PROBE), TP22.1 (PROBE), TP30.1 (PROBE), TP50.1 (PROBE), TP51.1 (PROBE), TP8.1 (PROBE)
- net ILIM: now also TP40.1 (PROBE)
- net IOREF_3V3: now also TP36.1 (PROBE)
- net OVLO: now also TP38.1 (PROBE)
- net PICO_3V3: now also TP35.1 (PROBE)
- net PICO_VSYS: now also TP34.1 (PROBE)
- net P_IO_OE_N: now also TP43.1 (PROBE)
- net P_SPI_MISO: now also TP46.1 (PROBE)
- net P_SPI_MOSI: now also TP45.1 (PROBE)
- net P_SPI_SCK: now also TP44.1 (PROBE)
- net RADIO_5V: now also TP1.1 (PROBE), TP15.1 (PROBE), TP23.1 (PROBE), TP32.1 (PROBE), TP9.1 (PROBE)
- net S1_BUSY: now also TP3.1 (PROBE)
- net S1_CS_N: now also TP2.1 (PROBE)
- net S1_IRQ: now also TP4.1 (PROBE)
- net S1_RESET_N: now also TP5.1 (PROBE)
- net S1_RX_EN: now also TP7.1 (PROBE)
- net S1_TX_EN: now also TP6.1 (PROBE)
- net S2_BUSY: now also TP11.1 (PROBE)
- net S2_CS_N: now also TP10.1 (PROBE)
- net S2_IRQ: now also TP12.1 (PROBE)
- net S2_RESET_N: now also TP13.1 (PROBE)
- net S3_BUSY: now also TP17.1 (PROBE)
- net S3_CS_N: now also TP16.1 (PROBE)
- net S3_IRQ: now also TP18.1 (PROBE)
- net S3_RESET_N: now also TP19.1 (PROBE)
- net S3_RX_EN: now also TP21.1 (PROBE)
- net S3_TX_EN: now also TP20.1 (PROBE)
- net S4_BUSY: now also TP25.1 (PROBE)
- net S4_CS_N: now also TP24.1 (PROBE)
- net S4_IRQ: now also TP26.1 (PROBE)
- net S4_RESET_N: now also TP27.1 (PROBE)
- net S4_RX_EN: now also TP29.1 (PROBE)
- net S4_TX_EN: now also TP28.1 (PROBE)
- net SPI_MISO: now also TP49.1 (PROBE)
- net SPI_MOSI: now also TP48.1 (PROBE)
- net SPI_SCK: now also TP47.1 (PROBE)
- net USB_VBUS: now also TP33.1 (PROBE)
- net UVLO: now also TP37.1 (PROBE)
Other:
- note added: "REV A LAYOUT REVIEW. NOT FOR FABRICATION."
- note removed: "REV A SCHEMATIC REVIEW. NO PCB LAYOUT OR FABRICATION RELEASE."
